File: VCU_tester.kicad_pcb (KiCad board)
At the start: 2 copper layers, 54.6 x 86.4 mm, 2 parts, among them P8 BeagleBone_Black_Header, P9 BeagleBone_Black_Header

Commit message: CAN parts added, rs232 parts added, gpio added
Connections:
- net Net-(P8-Pad10) renamed /GPIO_68
- net Net-(P8-Pad11) renamed /GPIO_45
- net Net-(P8-Pad12) renamed /GPIO_44
- net Net-(P8-Pad13) renamed /ETHRPWM2B
- net Net-(P8-Pad14) renamed /GPIO_26
- net Net-(P8-Pad15) renamed /GPIO_47
- net Net-(P8-Pad16) renamed /GPIO_46
- net Net-(P8-Pad17) renamed /GPIO_27
- net Net-(P8-Pad18) renamed /GPIO_65
- net Net-(P8-Pad19) renamed /ETHRPWM2A
- net Net-(P8-Pad20) renamed /MMC1_CMD
- net Net-(P8-Pad21) renamed /MMC1_CLK
- net Net-(P8-Pad22) renamed /MMC1_DAT5
- net Net-(P8-Pad23) renamed /MMC1_DAT4
- net Net-(P8-Pad24) renamed /MMC1_DAT1
- net Net-(P8-Pad25) renamed /MMC1_DATO
- net Net-(P8-Pad26) renamed /GPIO_61
- net Net-(P8-Pad27) renamed /LCD_VSYNC
- net Net-(P8-Pad28) renamed /LCD_PCLK
- net Net-(P8-Pad29) renamed /LCD_HSYNC
- net Net-(P8-Pad3) renamed /MMC1_DAT6
- net Net-(P8-Pad30) renamed /LCD_AC_BIAS
- net Net-(P8-Pad31) renamed /LCD_DATA14
- net Net-(P8-Pad32) renamed /LCD_DATA15
- net Net-(P8-Pad33) renamed /LCD_DATA13
- net Net-(P8-Pad34) renamed /LCD_DATA11
- net Net-(P8-Pad35) renamed /LCD_DATA12
- net Net-(P8-Pad36) renamed /LCD_DATA10
- net Net-(P8-Pad37) renamed /LCD_DATA8
- net Net-(P8-Pad38) renamed /LCD_DATA9
- net Net-(P8-Pad39) renamed /LCD_DATA6
- net Net-(P8-Pad4) renamed /MMC1_DAT7
- net Net-(P8-Pad40) renamed /LCD_DATA7
- net Net-(P8-Pad41) renamed /LCD_DATA4
- net Net-(P8-Pad42) renamed /LCD_DATA5
- net Net-(P8-Pad43) renamed /LCD_DATA2
- net Net-(P8-Pad44) renamed /LCD_DATA3
- net Net-(P8-Pad45) renamed /LCD_DATA0
- net Net-(P8-Pad46) renamed /LCD_DATA1
- net Net-(P8-Pad5) renamed /MMC1_DAT2
- net Net-(P8-Pad6) renamed /MMC1_DAT3
- net Net-(P8-Pad7) renamed /GPIO_66
- net Net-(P8-Pad8) renamed /GPIO_67
- net Net-(P8-Pad9) renamed /GPIO_69
- net Net-(P9-Pad11) renamed /UART4_RXD
- net Net-(P9-Pad12) renamed /GPIO_60
- net Net-(P9-Pad13) renamed /UART4_TXD
- net Net-(P9-Pad14) renamed /ETHRPWM1A
- net Net-(P9-Pad15) renamed /GPIO_48
- net Net-(P9-Pad16) renamed /ETHRPWM1B
- net Net-(P9-Pad17) renamed /SPIO_CSO
- net Net-(P9-Pad18) renamed /SPIO_D1
- net Net-(P9-Pad19) renamed /I2C2_SCL
- net Net-(P9-Pad20) renamed /I2C_SDA
- net Net-(P9-Pad21) renamed /SPIO_DO
- net Net-(P9-Pad22) renamed /SPIO_SCLK
- net Net-(P9-Pad23) renamed /GPIO_49
- net Net-(P9-Pad24) renamed /UART1_TXD
- net Net-(P9-Pad25) renamed /GPIO_117
- net Net-(P9-Pad26) renamed /UART1_RXD
- net Net-(P9-Pad27) renamed /GPIO_115
- net Net-(P9-Pad28) renamed /SP11_CSO
- net Net-(P9-Pad29) renamed /SP11_DO
- net Net-(P9-Pad30) renamed /GPIO_112
- net Net-(P9-Pad31) renamed /SP11_SCLK
- net Net-(P9-Pad33) renamed /AIN4
- net Net-(P9-Pad35) renamed /AIN6
- net Net-(P9-Pad36) renamed /AIN5
- net Net-(P9-Pad37) renamed /AIN2
- net Net-(P9-Pad38) renamed /AIN3
- net Net-(P9-Pad39) renamed /AIN0
- net Net-(P9-Pad40) renamed /AIN1
- net Net-(P9-Pad41) renamed /GPI0_20
- net Net-(P9-Pad42) renamed /ECAPWMO
