File: VCU_tester.kicad_pcb (KiCad board)
At the start: 2 copper layers, 240.2 x 171.8 mm, 101 parts, among them J1 Conn_01x04_Male, J10 DB9_Male, J11 DB9_Male, J12 Conn_01x08_Male, J13 Conn_01x08_Male, J14 USB_C_Receptacle, J2 Screw_Terminal_01x02, J3 DB9_Male, J4 DB9_Male, J5 DB9_Male, J500 Conn_01x08_Female, J501 Conn_01x08_Female, J502 Conn_01x08_Female, J504 Conn_02x18_Odd_Even, J505 Conn_01x10_Female, J506 Conn_01x08_Female, J507 Conn_01x08_Female, J6 DB9_Male, J7 Conn_01x04_Male, J8 DB9_Male, J9 DB9_Male, P8 BeagleBone_Black_Header, P9 BeagleBone_Black_Header, U1 REF3020, U2 MAX3232, U3 TCAN1042HVD, U4 MAX3232, U5 TCAN1042HVD, U6 DS3231MZ, U7 DS3231MZ

Commit message: cant remember what I added Im tired
Parts:
- added J15: USB_B_Micro, Connector_USB:USB_Micro-B_Molex-105017-0001, F.Cu at (202.5, 25.2)
- moved J14 0.28 mm to (191.1, 28.7)
Connections:
- BT1 pad 1: GNDD -> /RTC_VBAT
- BT1 pad 2: /RTC_VBAT -> GNDD
Routing:
- net Net-(J15-Pad6): track 0.00 -> 19.0 mm
- net +5V: track 219.8 -> 236.6 mm
- net GNDD: track 469.6 -> 482.1 mm
Other:
- board text added: "MAKE CUTOUT BIGGER FOR ETH"

Commit message: added comments
Other:
- board text added: "GET FOOTPRINT FOR VCU BOARD"
- board text added: "MAKE CUTOUT BIGGER FOR ETH?"
- board text removed: "MAKE CUTOUT BIGGER FOR ETH"
Changed lines of the file:
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@@
   (general
     (thickness 1.6)
-    (drawings 71)
+    (drawings 72)
     (tracks 672)
     (zones 0)
@@
     )
   )
-  (gr_text "MAKE CUTOUT BIGGER FOR ETH" (at 107.75 0) (layer F.Cu)
-    (effects (font (size 1.5 1.5) (thickness 0.3)))
+  (gr_text "GET FOOTPRINT FOR VCU BOARD" (at 326.4 114.9) (layer Dwgs.User)
+    (effects (font (size 5 5) (thickness 0.5)))
+  )
+  (gr_text "MAKE CUTOUT BIGGER FOR ETH?" (at 107.75 0) (layer Dwgs.User)
+    (effects (font (size 5 5) (thickness 0.5)))
   )
   (gr_line (start 254.5 22.5) (end 260 194) (layer Edge.Cuts) (width 0.00254))

Commit message: placed vcu and beaglebone
Parts:
- removed J10: DB9_Male, Connector_Dsub:DSUB-9_Male_Horizontal_P2.77x2.84mm_EdgePinOffset7.70mm_Housed_MountingHolesOffset9.12mm
- removed J506: Conn_01x08_Female, Connector_PinSocket_2.54mm:PinSocket_1x08_P2.54mm_Vertical
- added J503: Conn_01x08_Female, Connector_PinSocket_2.54mm:PinSocket_1x08_P2.54mm_Vertical, F.Cu at (358.1, 66.0)
- added REF**: BeagleBone-Black_Flip, project:BeagleBone-Black_Flip, F.Cu at (457.2, 50.8)
- added REF**: SAME70-XPLD_Flip, project:SAME70-XPLD_Flip, F.Cu at (309.9, 101.6)
- J500: value Conn_01x08_Female -> Conn_01x10_Female; footprint Connector_PinSocket_2.54mm:PinSocket_1x08_P2.54mm_Vertical -> Connector_PinSocket_2.54mm:PinSocket_1x10_P2.54mm_Vertical
- J504: value Conn_02x18_Odd_Even -> Conn_01x08_Female; footprint Connector_PinSocket_2.54mm:PinSocket_2x18_P2.54mm_Vertical -> Connector_PinSocket_2.54mm:PinSocket_1x08_P2.54mm_Vertical
- J505: value Conn_01x10_Female -> Conn_01x08_Female; footprint Connector_PinSocket_2.54mm:PinSocket_1x10_P2.54mm_Vertical -> Connector_PinSocket_2.54mm:PinSocket_1x08_P2.54mm_Vertical
- J507: value Conn_01x08_Female -> Conn_02x18_Odd_Even; footprint Connector_PinSocket_2.54mm:PinSocket_1x08_P2.54mm_Vertical -> Connector_PinSocket_2.54mm:PinSocket_2x18_P2.54mm_Vertical
- P8, P9: footprint Socket_BeagleBone_Black:Socket_BeagleBone_Black -> project:PinHeader_2x23_P2.54mm_Vertical_Flip
- moved P9 398.0 mm to (457.2, 50.8)
- moved P8 302.0 mm to (408.9, 50.8)
- moved J505 232.7 mm to (358.1, 43.2), turned to 0 degrees
- moved J500 212.5 mm to (358.1, 87.9), turned to 0 degrees
- moved J14 197.7 mm to (388.6, 36.6)
- moved J15 196.4 mm to (398.8, 33.1)
- moved J507 190.7 mm to (358.1, 35.6), turned to 270 degrees
- moved J501 139.1 mm to (309.9, 101.6), turned to 180 degrees
- moved J502 116.3 mm to (309.9, 78.7), turned to 180 degrees
- moved J504 91.2 mm to (309.9, 55.9), turned to 180 degrees
Connections:
- J11 pad 1: Net-(J11-Pad1) -> (no net)
- J11 pad 4: Net-(J11-Pad4) -> (no net)
- J11 pad 5: Net-(J11-Pad5) -> (no net)
- J11 pad 6: Net-(J11-Pad6) -> (no net)
- J11 pad 7: Net-(J11-Pad7) -> (no net)
- J11 pad 8: Net-(J11-Pad8) -> (no net)
- J11 pad 9: Net-(J11-Pad9) -> (no net)
- J14 pad A5: Net-(J14-PadA5) -> (no net)
- J14 pad A6: Net-(J14-PadA6) -> (no net)
- J14 pad A7: Net-(J14-PadA7) -> (no net)
- J14 pad A8: Net-(J14-PadA8) -> (no net)
- J14 pad B5: Net-(J14-PadB5) -> (no net)
- J14 pad B6: Net-(J14-PadB6) -> (no net)
- J14 pad B7: Net-(J14-PadB7) -> (no net)
- J14 pad B8: Net-(J14-PadB8) -> (no net)
- J15 pad 2: Net-(J15-Pad2) -> (no net)
- J15 pad 3: Net-(J15-Pad3) -> (no net)
- J15 pad 4: Net-(J15-Pad4) -> (no net)
- J3 pad 1: Net-(J3-Pad1) -> (no net)
- J3 pad 2: Net-(J3-Pad2) -> (no net)
- J3 pad 5: Net-(J3-Pad5) -> (no net)
- J3 pad 6: Net-(J3-Pad6) -> (no net)
- J3 pad 7: Net-(J3-Pad7) -> (no net)
- J3 pad 9: Net-(J3-Pad9) -> (no net)
- J4 pad 1: Net-(J4-Pad1) -> (no net)
- J4 pad 2: Net-(J4-Pad2) -> (no net)
- J4 pad 5: Net-(J4-Pad5) -> (no net)
- J4 pad 6: Net-(J4-Pad6) -> (no net)
- J4 pad 7: Net-(J4-Pad7) -> (no net)
- J4 pad 9: Net-(J4-Pad9) -> (no net)
- J5 pad 1: Net-(J5-Pad1) -> (no net)
- J5 pad 2: Net-(J5-Pad2) -> (no net)
- J5 pad 5: Net-(J5-Pad5) -> (no net)
- J5 pad 6: Net-(J5-Pad6) -> (no net)
- J5 pad 7: Net-(J5-Pad7) -> (no net)
- J5 pad 9: Net-(J5-Pad9) -> (no net)
- J500 pad 1: Net-(J500-Pad1) -> (no net)
- J500 pad 2: +3.3VA -> /GPIO_4
- J500 pad 3: /GPIO_112 -> /VCUGPIO_10
- J500 pad 4: +3.3VA -> (no net)
- J500 pad 5: +5V -> (no net)
- J500 pad 6: GNDD -> (no net)
- J500 pad 8: +5V -> /VCU_REFVOLT
- J501 pad 1: /VCUGPIO_10 -> (no net)
- J501 pad 2: /TempRin -> +3.3VA
- J501 pad 3: /PressRout -> /GPIO_112
- J501 pad 4: /PressRin -> +3.3VA
- J501 pad 5: /TempRout -> +5V
- J501 pad 6: /TempLout -> GNDD
- J501 pad 7: Net-(J501-Pad7) -> GNDD
- J501 pad 8: /TempLin -> +5V
- J502 pad 1: Net-(J502-Pad1) -> /VCUGPIO_10
- J502 pad 2: Net-(J502-Pad2) -> /TempRin
- J502 pad 3: Net-(J502-Pad3) -> /PressRout
- J502 pad 4: Net-(J502-Pad4) -> /PressRin
- J502 pad 5: Net-(J502-Pad5) -> /TempRout
- J502 pad 6: Net-(J502-Pad6) -> /TempLout
- J502 pad 7: /VCUCANRX0 -> (no net)
- J502 pad 8: /VCUCANTX0 -> /TempLin
- J504 pad 1: +5V -> (no net)
- J504 pad 2: +5V -> (no net)
- J504 pad 3: /GPIO_44 -> (no net)
- J504 pad 4: /GPIO_45 -> (no net)
- J504 pad 5: /GPIO_46 -> (no net)
- J504 pad 6: /GPIO_47 -> (no net)
- J504 pad 7: /GPIO_48 -> /VCUCANRX0
- J504 pad 8: /GPIO_49 -> /VCUCANTX0
- J505 pad 1: /VCUGPIO_8 -> /PD28
- J505 pad 2: /GPIO_4 -> /PD27
- J505 pad 3: /VCUGPIO_10 -> (no net)
- J505 pad 4: /VCUGPIO_11 -> (no net)
- J505 pad 5: /VCUGPIO_12 -> (no net)
- J505 pad 6: Net-(J505-Pad6) -> (no net)
- J505 pad 7: GNDD -> (no net)
- J505 pad 8: /VCU_REFVOLT -> (no net)
- J507 pad 1: /PD28 -> +5V
- J507 pad 2: /PD27 -> +5V
- J507 pad 3: /VCURXD4 -> /GPIO_44
- J507 pad 4: /VCUTXD4 -> /GPIO_45
- J507 pad 5: /VCURXD2 -> /GPIO_46
- J507 pad 6: /VCUTXD2 -> /GPIO_47
- J507 pad 7: /VCURXD0 -> /GPIO_48
- J507 pad 8: /VCUTXD0 -> /GPIO_49
- J6 pad 1: Net-(J6-Pad1) -> (no net)
- J6 pad 2: Net-(J6-Pad2) -> (no net)
- J6 pad 5: Net-(J6-Pad5) -> (no net)
- J6 pad 6: Net-(J6-Pad6) -> (no net)
- J6 pad 7: Net-(J6-Pad7) -> (no net)
- J6 pad 9: Net-(J6-Pad9) -> (no net)
- J8 pad 1: Net-(J8-Pad1) -> (no net)
- J8 pad 4: Net-(J8-Pad4) -> (no net)
- J8 pad 5: Net-(J8-Pad5) -> (no net)
- J8 pad 6: Net-(J8-Pad6) -> (no net)
- J8 pad 7: Net-(J8-Pad7) -> (no net)
- J8 pad 8: Net-(J8-Pad8) -> (no net)
- J8 pad 9: Net-(J8-Pad9) -> (no net)
- J9 pad 1: Net-(J9-Pad1) -> (no net)
- J9 pad 4: Net-(J9-Pad4) -> (no net)
- J9 pad 5: Net-(J9-Pad5) -> (no net)
- J9 pad 6: Net-(J9-Pad6) -> (no net)
- J9 pad 7: Net-(J9-Pad7) -> (no net)
- J9 pad 8: Net-(J9-Pad8) -> (no net)
- J9 pad 9: Net-(J9-Pad9) -> (no net)
- P8 pad 13: /GPIO_23 -> (no net)
- P8 pad 14: /GPIO_26 -> (no net)
- P8 pad 17: /GPIO_27 -> (no net)
- P8 pad 20: /GPIO_63 -> (no net)
- P8 pad 21: /GPIO_62 -> (no net)
- P8 pad 22: /GPIO_37 -> (no net)
- P8 pad 23: /GPIO_36 -> (no net)
- P8 pad 24: /GPIO_33 -> (no net)
- P8 pad 25: /GPIO_32 -> (no net)
- P8 pad 27: /GPIO_86 -> (no net)
- P8 pad 28: /GPIO_88 -> (no net)
- P8 pad 29: /GPIO_87 -> (no net)
- P8 pad 3: /MMC1_Dat6 -> (no net)
- P8 pad 30: /GPIO_89 -> (no net)
- P8 pad 31: /UART5_CSTN+ -> (no net)
- P8 pad 32: /UART5_RTSN -> (no net)
- P8 pad 33: /UART4_RSTN -> (no net)
- P8 pad 34: /UART3_RTSN -> (no net)
- P8 pad 35: /UART4_CTSN -> (no net)
- P8 pad 36: /UART3_CTSN -> (no net)
- P8 pad 37: /UART5_TXD+ -> (no net)
- P8 pad 38: /UART5_RXD+ -> (no net)
- P8 pad 39: /GPIO_76 -> (no net)
- P8 pad 4: /MMC1_dat7 -> (no net)
- P8 pad 40: /GPIO_77 -> (no net)
- P8 pad 41: /GPIO_74 -> (no net)
- P8 pad 42: /GPIO_75 -> (no net)
- P8 pad 43: /GPIO_72 -> (no net)
- P8 pad 44: /GPIO_73 -> (no net)
- P8 pad 45: /GPIO_70 -> (no net)
- P8 pad 46: /GPIO_71 -> (no net)
- P8 pad 5: /MMC1_Dat2 -> (no net)
- P8 pad 6: /MMC1_dat3 -> (no net)
- P8 pad 8: /GPIO_67 -> (no net)
- P9 pad 28: /SPI1_CSO -> (no net)
- P9 pad 29: /SPI1_DO -> (no net)
- P9 pad 31: /SPI1_SCLK -> (no net)
- P9 pad 32: VDD_ADC -> (no net)
- P9 pad 33: /AIN4 -> (no net)
- P9 pad 34: GNDA_ADC -> (no net)
- P9 pad 35: /AIN6 -> (no net)
- P9 pad 36: /AIN5 -> (no net)
- P9 pad 37: /AIN2 -> (no net)
- P9 pad 38: /AIN3 -> (no net)
- P9 pad 39: /AIN0 -> (no net)
- P9 pad 40: /AIN1 -> (no net)
- P9 pad 41: /GPI0_20 -> (no net)
- P9 pad 42: /UART3_TXD -> (no net)
- U6 pad 1: Net-(U6-Pad1) -> (no net)
- U6 pad 3: Net-(U6-Pad3) -> (no net)
- U6 pad 4: Net-(U6-Pad4) -> (no net)
- U7 pad 1: Net-(U7-Pad1) -> (no net)
- U7 pad 3: Net-(U7-Pad3) -> (no net)
- U7 pad 4: Net-(U7-Pad4) -> (no net)
Other:
- board size 240.2 x 171.8 mm -> 203.2 x 25.4 mm
- board text added: "178-009-613R491"
- board text removed: "GET FOOTPRINT FOR VCU BOARD"

Commit message: new, compact (and sexy) design
Parts:
- removed the REF** at (457.2, 50.8)
- added J10: DB9_Male, Connector_Dsub:DSUB-9_Male_Vertical_P2.77x2.84mm_MountingHoles, F.Cu at (145.0, 0.00)
- added JP10: Jumper, Connector_PinHeader_2.00mm:PinHeader_1x03_P2.00mm_Vertical, F.Cu at (106.0, 26.5)
- added JP11: Jumper, Connector_PinHeader_2.00mm:PinHeader_1x03_P2.00mm_Vertical, F.Cu at (96.0, 26.5)
- added JP12: Jumper, Connector_PinHeader_2.00mm:PinHeader_1x03_P2.00mm_Vertical, F.Cu at (111.0, 26.5)
- added JP13: Jumper_3_Bridged12, Connector_PinHeader_2.00mm:PinHeader_1x03_P2.00mm_Vertical, F.Cu at (123.0, 4.00)
- added JP14: Jumper_3_Bridged12, Connector_PinHeader_2.00mm:PinHeader_1x03_P2.00mm_Vertical, F.Cu at (128.5, 4.00)
- added JP15: Jumper_3_Bridged12, Connector_PinHeader_2.00mm:PinHeader_1x03_P2.00mm_Vertical, F.Cu at (163.0, 4.00)
- added JP16: Jumper_3_Bridged12, Connector_PinHeader_2.00mm:PinHeader_1x03_P2.00mm_Vertical, F.Cu at (168.0, 4.00)
- added JP9: Jumper_3_Bridged12, Connector_PinHeader_2.00mm:PinHeader_1x03_P2.00mm_Vertical, F.Cu at (48.0, 5.00)
- added REF**: BeagleBone-Black, project:BeagleBone-Black, F.Cu at (65.0, 80.0)
- J11, J3, J4, J5, J6, J8, J9: footprint Connector_Dsub:DSUB-9_Male_Horizontal_P2.77x2.84mm_EdgePinOffset7.70mm_Housed_MountingHolesOffset9.12mm -> Connector_Dsub:DSUB-9_Male_Vertical_P2.77x2.84mm_MountingHoles
- JP5, JP6, JP7: value Jumper -> Jumper_3_Bridged12
- P8, P9: footprint project:PinHeader_2x23_P2.54mm_Vertical_Flip -> Socket_BeagleBone_Black:Socket_BeagleBone_Black
- moved J15 398.8 mm to (0.14, 42.5), turned to 270 degrees
- moved P9 393.3 mm to (65.0, 80.0)
- moved J14 385.4 mm to (3.60, 53.9), turned to 270 degrees
- moved P8 297.1 mm to (113.2, 80.0)
- moved J500 168.4 mm to (190.6, 105.4)
- moved J501 168.4 mm to (142.4, 119.1)
- moved J502 168.4 mm to (142.4, 96.2)
- moved J503 168.4 mm to (190.6, 83.5)
- moved J504 168.4 mm to (142.4, 73.4)
- moved J505 168.4 mm to (190.6, 60.7)
- moved J507 168.4 mm to (190.6, 53.1)
- moved REF** 168.4 mm to (142.4, 119.1)
- moved J13 117.1 mm to (37.5, 60.0), turned to 0 degrees
- moved TP46 114.2 mm to (187.5, 20.0), turned to 0 degrees
- moved J2 110.0 mm to (127.6, -12.5), turned to 180 degrees
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Connections:
- J11 pad 1: (no net) -> Net-(J11-Pad1)
- J11 pad 2: /motor_controller/VRRX -> Net-(J11-Pad2)
- J11 pad 3: /motor_controller/VRTX -> Net-(J11-Pad3)
- J11 pad 4: (no net) -> Net-(J11-Pad4)
- J11 pad 5: (no net) -> Net-(J11-Pad5)
- J11 pad 6: (no net) -> Net-(J11-Pad6)
- J11 pad 7: (no net) -> Net-(J11-Pad7)
- J11 pad 8: (no net) -> Net-(J11-Pad8)
- J11 pad 9: (no net) -> Net-(J11-Pad9)
- J14 pad A5: (no net) -> Net-(J14-PadA5)
- J14 pad A6: (no net) -> Net-(J14-PadA6)
- J14 pad A7: (no net) -> Net-(J14-PadA7)
- J14 pad A8: (no net) -> Net-(J14-PadA8)
- J14 pad B5: (no net) -> Net-(J14-PadB5)
- J14 pad B6: (no net) -> Net-(J14-PadB6)
- J14 pad B7: (no net) -> Net-(J14-PadB7)
- J14 pad B8: (no net) -> Net-(J14-PadB8)
- J15 pad 2: (no net) -> Net-(J15-Pad2)
- J15 pad 3: (no net) -> Net-(J15-Pad3)
- J15 pad 4: (no net) -> Net-(J15-Pad4)
- J3 pad 1: (no net) -> Net-(J3-Pad1)
- J3 pad 2: (no net) -> Net-(J3-Pad2)
- J3 pad 5: (no net) -> Net-(J3-Pad5)
- J3 pad 6: (no net) -> Net-(J3-Pad6)
- J3 pad 7: (no net) -> Net-(J3-Pad7)
- J3 pad 9: (no net) -> Net-(J3-Pad9)
- J4 pad 1: (no net) -> Net-(J4-Pad1)
- J4 pad 2: (no net) -> Net-(J4-Pad2)
- J4 pad 5: (no net) -> Net-(J4-Pad5)
- J4 pad 6: (no net) -> Net-(J4-Pad6)
- J4 pad 7: (no net) -> Net-(J4-Pad7)
- J4 pad 9: (no net) -> Net-(J4-Pad9)
- J5 pad 1: (no net) -> Net-(J5-Pad1)
- J5 pad 2: (no net) -> Net-(J5-Pad2)
- J5 pad 5: (no net) -> Net-(J5-Pad5)
- J5 pad 6: (no net) -> Net-(J5-Pad6)
- J5 pad 7: (no net) -> Net-(J5-Pad7)
- J5 pad 9: (no net) -> Net-(J5-Pad9)
- J500 pad 1: (no net) -> /VCUGPIO_8
- J500 pad 10: (no net) -> Net-(J500-Pad10)
- J500 pad 4: (no net) -> /VCUGPIO_11
- J500 pad 5: (no net) -> /VCUGPIO_12
- J500 pad 6: (no net) -> Net-(J500-Pad6)
- J500 pad 9: (no net) -> Net-(J500-Pad9)
- J501 pad 1: (no net) -> Net-(J501-Pad1)
- J502 pad 7: (no net) -> Net-(J502-Pad7)
- J503 pad 5: (no net) -> /VCUGPIO_4
- J503 pad 6: (no net) -> /VCUGPIO_5
- J504 pad 1: (no net) -> Net-(J504-Pad1)
- J504 pad 2: (no net) -> Net-(J504-Pad2)
- J504 pad 3: (no net) -> Net-(J504-Pad3)
- J504 pad 4: (no net) -> Net-(J504-Pad4)
- J504 pad 5: (no net) -> Net-(J504-Pad5)
- J504 pad 6: (no net) -> Net-(J504-Pad6)
- J505 pad 3: (no net) -> /VCURXD4
- J505 pad 4: (no net) -> /VCUTXD4
- J505 pad 5: (no net) -> /VCURXD2
- J505 pad 6: (no net) -> /VCUTXD2
- J505 pad 7: (no net) -> /VCURXD0
- J505 pad 8: (no net) -> /VCUTXD0
- J507 pad 11: (no net) -> Net-(J507-Pad11)
- J507 pad 12: (no net) -> Net-(J507-Pad12)
- J507 pad 13: (no net) -> Net-(J507-Pad13)
- J507 pad 14: (no net) -> Net-(J507-Pad14)
- J507 pad 15: (no net) -> Net-(J507-Pad15)
- J507 pad 16: (no net) -> Net-(J507-Pad16)
- J507 pad 17: (no net) -> Net-(J507-Pad17)
- J507 pad 18: (no net) -> Net-(J507-Pad18)
- J507 pad 19: (no net) -> Net-(J507-Pad19)
- J507 pad 20: (no net) -> Net-(J507-Pad20)
- J507 pad 21: (no net) -> Net-(J507-Pad21)
- J507 pad 22: (no net) -> Net-(J507-Pad22)
- J507 pad 23: (no net) -> Net-(J507-Pad23)
- J507 pad 24: (no net) -> Net-(J507-Pad24)
- J507 pad 25: (no net) -> Net-(J507-Pad25)
- J507 pad 26: (no net) -> Net-(J507-Pad26)
- J507 pad 28: (no net) -> /VCUTXD1
- J507 pad 29: (no net) -> /AIR3
- J507 pad 30: (no net) -> /AIR2
- J507 pad 32: (no net) -> /AIR1
- J507 pad 33: (no net) -> /VCUCANRX1
- J6 pad 1: (no net) -> Net-(J6-Pad1)
- J6 pad 2: (no net) -> Net-(J6-Pad2)
- J6 pad 5: (no net) -> Net-(J6-Pad5)
- J6 pad 6: (no net) -> Net-(J6-Pad6)
- J6 pad 7: (no net) -> Net-(J6-Pad7)
- J6 pad 9: (no net) -> Net-(J6-Pad9)
- J8 pad 1: (no net) -> Net-(J8-Pad1)
- J8 pad 2: /motor_controller/BBLRX -> Net-(J8-Pad2)
- J8 pad 3: /motor_controller/BBLTX -> Net-(J8-Pad3)
- J8 pad 4: (no net) -> Net-(J8-Pad4)
- J8 pad 5: (no net) -> Net-(J8-Pad5)
- J8 pad 6: (no net) -> Net-(J8-Pad6)
- J8 pad 7: (no net) -> Net-(J8-Pad7)
- J8 pad 8: (no net) -> Net-(J8-Pad8)
- J8 pad 9: (no net) -> Net-(J8-Pad9)
- J9 pad 1: (no net) -> Net-(J9-Pad1)
- J9 pad 2: /motor_controller/BBRRX -> Net-(J9-Pad2)
- J9 pad 3: /motor_controller/BBRTX -> Net-(J9-Pad3)
- J9 pad 4: (no net) -> Net-(J9-Pad4)
- J9 pad 5: (no net) -> Net-(J9-Pad5)
- J9 pad 6: (no net) -> Net-(J9-Pad6)
- J9 pad 7: (no net) -> Net-(J9-Pad7)
- J9 pad 8: (no net) -> Net-(J9-Pad8)
- J9 pad 9: (no net) -> Net-(J9-Pad9)
- JP5 pad 1: /motor_controller/BBLTX -> Net-(J8-Pad3)
- JP5 pad 2: /motor_controller/VLTX -> /motor_controller/BBRTX
- JP5 pad 3: (no net) -> Net-(J8-Pad2)
- JP6 pad 1: /motor_controller/BBLRX -> Net-(J8-Pad2)
- JP6 pad 2: /motor_controller/VLRX -> /motor_controller/BBRRX
- JP6 pad 3: (no net) -> Net-(J8-Pad3)
- JP7 pad 1: /motor_controller/BBRTX -> Net-(J9-Pad3)
- JP7 pad 2: /motor_controller/VRTX -> /motor_controller/BBLTX
- JP7 pad 3: (no net) -> Net-(J9-Pad2)
- JP8 pad 1: /motor_controller/BBRRX -> Net-(J9-Pad2)
- JP8 pad 2: /motor_controller/VRRX -> Net-(J11-Pad2)
- P8 pad 13: (no net) -> /GPIO_23
- P8 pad 14: (no net) -> /GPIO_26
- P8 pad 17: (no net) -> /GPIO_27
- P8 pad 20: (no net) -> /GPIO_63
- P8 pad 21: (no net) -> /GPIO_62
- P8 pad 22: (no net) -> /GPIO_37
- P8 pad 23: (no net) -> /GPIO_36
- P8 pad 24: (no net) -> /GPIO_33
- P8 pad 25: (no net) -> /GPIO_32
- P8 pad 27: (no net) -> /GPIO_86
- P8 pad 28: (no net) -> /GPIO_88
- P8 pad 29: (no net) -> /GPIO_87
- P8 pad 3: (no net) -> /MMC1_Dat6
- P8 pad 30: (no net) -> /GPIO_89
- P8 pad 31: (no net) -> /UART5_CSTN+
- P8 pad 32: (no net) -> /UART5_RTSN
- P8 pad 33: (no net) -> /UART4_RSTN
- P8 pad 34: (no net) -> /UART3_RTSN
- P8 pad 35: (no net) -> /UART4_CTSN
- P8 pad 36: (no net) -> /UART3_CTSN
- P8 pad 37: (no net) -> /UART5_TXD+
- P8 pad 38: (no net) -> /UART5_RXD+
- P8 pad 39: (no net) -> /GPIO_76
- P8 pad 4: (no net) -> /MMC1_dat7
- P8 pad 40: (no net) -> /GPIO_77
- P8 pad 41: (no net) -> /GPIO_74
- P8 pad 42: (no net) -> /GPIO_75
- P8 pad 43: (no net) -> /GPIO_72
- P8 pad 44: (no net) -> /GPIO_73
- P8 pad 45: (no net) -> /GPIO_70
- P8 pad 46: (no net) -> /GPIO_71
- P8 pad 5: (no net) -> /MMC1_Dat2
- P8 pad 6: (no net) -> /MMC1_dat3
- P8 pad 8: (no net) -> /GPIO_67
- P9 pad 28: (no net) -> /SPI1_CSO
- P9 pad 29: (no net) -> /SPI1_DO
- P9 pad 31: (no net) -> /SPI1_SCLK
- P9 pad 32: (no net) -> VDD_ADC
- P9 pad 33: (no net) -> /AIN4
- P9 pad 34: (no net) -> GNDA_ADC
- P9 pad 35: (no net) -> /AIN6
- P9 pad 36: (no net) -> /AIN5
- P9 pad 37: (no net) -> /AIN2
- P9 pad 38: (no net) -> /AIN3
- P9 pad 39: (no net) -> /AIN0
- P9 pad 40: (no net) -> /AIN1
- P9 pad 41: (no net) -> /GPI0_20
- P9 pad 42: (no net) -> /UART3_TXD
- U6 pad 1: (no net) -> Net-(U6-Pad1)
- U6 pad 3: (no net) -> Net-(U6-Pad3)
- U6 pad 4: (no net) -> Net-(U6-Pad4)
- U7 pad 1: (no net) -> Net-(U7-Pad1)
- U7 pad 3: (no net) -> Net-(U7-Pad3)
- U7 pad 4: (no net) -> Net-(U7-Pad4)
Routing:
- net GNDD: track 482.1 -> 196.0 mm, vias 0 -> 1
- net +5V: track 236.6 -> 44.2 mm
- net Net-(J9-Pad3): track 0.00 -> 89.2 mm
- net Net-(J9-Pad2): track 0.00 -> 80.6 mm
- net +3.3VA: track 84.6 -> 13.3 mm, vias 1 -> 0
- net +3V3: track 112.2 -> 47.2 mm
- net VCUCAN+: track 125.9 -> 70.4 mm, vias 3 -> 1
- net VCUCAN-: track 120.8 -> 66.0 mm
- net Net-(J8-Pad3): track 0.00 -> 54.2 mm
- net BBCAN+: track 125.9 -> 75.3 mm
- net Net-(J8-Pad2): track 0.00 -> 50.5 mm, vias 0 -> 1
- net BBCAN-: track 132.8 -> 90.6 mm
- net /motor_controller/VLRX: track 90.5 -> 51.1 mm
- net /motor_controller/VLTX: track 71.9 -> 41.0 mm
- net /motor_controller/BBRTX: track 57.8 -> 27.4 mm
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Other:
- board size 203.2 x 25.4 mm -> 200 x 172.5 mm
- board text added: "BB RS232 L"
- board text added: "BB RS232 R"
- board text added: "BB UART1"
- board text added: "VCU RS232 L"
- board text added: "VCU RS232 R"
- board text removed: "MAKE CUTOUT BIGGER FOR ETH?"
