File: motor_controller_uart.sch (KiCad schematic (older format))
At the start: 2 parts, among them U1 MAX232, U2 MAX232

Commit message: added vcu pinout, still lots needs doing
Parts:
- removed U1, U2: MAX232, symbol Interface_UART:MAX232
Changed lines of the file:
@@
 Comment4 ""
 $EndDescr
-$Comp
-L Interface_UART:MAX232 U?
-U 1 1 5ED8EA5F
-P 4800 3550
-AR Path="/5ED8EA5F" Ref="U?"  Part="1"
-AR Path="/5ED7E94C/5ED8EA5F" Ref="U1"  Part="1"
-F 0 "U1" H 4800 4931 50  0000 C CNN
-F 1 "MAX232" H 4800 4840 50  0000 C CNN
-F 2 "" H 4850 2500 50  0001 L CNN
-F 3 "http://www.ti.com/lit/ds/symlink/max232.pdf" H 4800 3650 50  0001 C CNN
-	1    4800 3550
-	1    0    0    -1
-$EndComp
-$Comp
-L Interface_UART:MAX232 U?
-U 1 1 5ED8EA65
-P 7400 3550
-AR Path="/5ED8EA65" Ref="U?"  Part="1"
-AR Path="/5ED7E94C/5ED8EA65" Ref="U2"  Part="1"
-F 0 "U2" H 7400 4931 50  0000 C CNN
-F 1 "MAX232" H 7400 4840 50  0000 C CNN
-F 2 "" H 7450 2500 50  0001 L CNN
-F 3 "http://www.ti.com/lit/ds/symlink/max232.pdf" H 7400 3650 50  0001 C CNN
-	1    7400 3550
-	1    0    0    -1
-$EndComp
 $EndSCHEMATC

Commit message: added pin names vcu, rs232 mcguffins, losing hope
Parts:
- added C17, C19, C20, C21, C23, C24: 0.1u, symbol Device:C_Small
- added C18, C22: C, symbol Device:C
- added J10, J11, J8, J9: DB9_Male, symbol Connector:DB9_Male
- added TP24, TP25, TP26, TP27, TP28, TP29, TP30, TP31, TP32, TP33, TP34, TP35, TP36, TP37, TP38, TP39: TestPoint, symbol Connector:TestPoint
- added U2, U4: MAX3232, symbol Interface_UART:MAX3232
Connections:
- new net: C17.1, U2.1 (C1+)
- new net: J8.2, TP30.1, U2.13 (R1IN)
- new net: J8.3, TP28.1, U2.14 (T1OUT)
- new net: C20.2, U2.2 (VS+)
- new net: C17.2, U2.3 (C1-)
- new net: C19.2, U2.4 (C2+)
- new net: C19.1, U2.5 (C2-)
- new net: C20.1, U2.6 (VS-)
- new net: J9.3, TP29.1, U2.7 (T2OUT)
- new net: J9.2, TP31.1, U2.8 (R2IN)
- new net: C21.1, U4.1 (C1+)
- new net: J10.2, TP38.1, U4.13 (R1IN)
- new net: J10.3, TP36.1, U4.14 (T1OUT)
- new net: C24.2, U4.2 (VS+)
- new net: C21.2, U4.3 (C1-)
- new net: C23.2, U4.4 (C2+)
- new net: C23.1, U4.5 (C2-)
- new net: C24.1, U4.6 (VS-)
- new net: J11.3, TP37.1, U4.7 (T2OUT)
- new net: J11.2, TP39.1, U4.8 (R2IN)
- new net +3V3: C18.1, C22.1, U2.16 (VCC), U4.16 (VCC)
- new net BBLR: TP26.1, U2.12 (R1OUT)
- new net BBLT: TP24.1, U2.11 (T1IN)
- new net BBRR: TP27.1, U2.9 (R2OUT)
- new net BBRT: TP25.1, U2.10 (T2IN)
- new net GNDD: C18.2, C22.2, U2.15 (GND), U4.15 (GND)
- new net VCULR: TP34.1, U4.12 (R1OUT)
- new net VCULT: TP32.1, U4.11 (T1IN)
- new net VCURR: TP35.1, U4.9 (R2OUT)
- new net VCURT: TP33.1, U4.10 (T2IN)
- no-connect marks 0 -> 28
